File: CMOSworkshop/4051.sch (KiCad schematic (older format))
At the start: 5 parts, among them U2 4051

Commit message: TRACE LAYOUT
Changed lines of the file:
@@
 Wire Wire Line
 	7200 2450 7000 2450
+Connection ~ 7000 3300
+Connection ~ 5600 3500
 $EndSCHEMATC
