File: CMOSworkshop/CMOSworkshop.kicad_pcb (KiCad board)
At the start: 2 copper layers, 127 x 76.2 mm, 73 parts, among them J1 JACK_STEREO, P1 CLK, P10 CLKSA&B, P11 OUTS, P12 OUTS, P3 OUTS, P5 MIX_IN, P6 CLKS/INH, P8 STEP OUT, SW1 SW_DPDT_x2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

Commit message: TRACE LAYOUT
Parts:
- removed C12: 10uF, Capacitors_ThroughHole:C_Radial_D5_L6_P2.5
- added REF**: touchpad, touchpad2, F.Cu at (159.0, 107.4)
- added REF**: touchpad, touchpad2, F.Cu at (138.0, 107.3)
- added REF**: touchpad, touchpad2, F.Cu at (148.3, 111.7)
- added REF**: touchpad, touchpad2, F.Cu at (116.9, 108.1)
- added REF**: touchpad, touchpad2, F.Cu at (127.6, 111.2)
- added REF**: touchpad, touchpad2, F.Cu at (106.3, 111.2)
- moved C7 7.91 mm to (187.2, 99.1), turned to 0 degrees
- moved R1 7.54 mm to (109.2, 84.2)
- moved R2 7.41 mm to (116.7, 84.2)
- moved C16 2.73 mm to (104.9, 91.5), turned to 270 degrees
- moved R10 2.64 mm to (188.5, 101.6)
- moved C15 2.62 mm to (183.9, 91.5), turned to 270 degrees
- moved R4 2.61 mm to (111.7, 84.2)
- moved C18 2.58 mm to (81.2, 91.7), turned to 270 degrees
- moved C17 2.58 mm to (131.3, 91.6), turned to 270 degrees
- moved C19 2.54 mm to (197.5, 91.4), turned to 270 degrees
- moved C14 2.46 mm to (157.5, 91.6), turned to 270 degrees
- moved R3 2.43 mm to (114.3, 84.2)
- moved P1 0.97 mm to (153.0, 82.8)
- moved R5 0.82 mm to (154.5, 85.8)
- moved RV7 0.75 mm to (173.8, 63.1)
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Connections:
- U1 pad 7: VCC -> GND
- U2 pad 8: VCC -> GND
Routing:
- net GND: track 0.00 -> 182.4 mm
- net VCC: track 0.00 -> 62.4 mm
- net inhibit: track 0.00 -> 36.6 mm
- net CLKB: track 0.00 -> 32.3 mm
- net q5: track 0.00 -> 22.7 mm
- net clkC: track 0.00 -> 21.2 mm
- net inC: track 0.00 -> 19.6 mm
- net Net-(C10-Pad-): track 0.00 -> 18.2 mm
- net Net-(C7-Pad2): track 0.00 -> 18.2 mm
- net q4: track 0.00 -> 17.2 mm
- net Net-(D2-Pad2): track 0.00 -> 16.4 mm
- net CLKA: track 0.00 -> 16.3 mm
- net q11: track 0.00 -> 15.0 mm
- net Q3B: track 0.00 -> 14.9 mm
- net Q1B: track 0.00 -> 14.2 mm
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