File: CMOSworkshop/CMOSworkshop_ThinStrips.sch (KiCad schematic (older format))
At the start: 38 parts, among them P1 CONN_01X03, P10 CONN_01X02, P11 CONN_01X03, P12 CONN_01X02, P13 CONN_01X03, P14 CONN_01X02, P15 CONN_01X03, P16 CONN_01X02, P17 CONN_01X02, P18 MIX_IN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

Commit message: added traces for mixer circuit and made small connection in hp mixer
Parts:
- RV1, RV2, RV3, RV4, RV5, RV6: symbol POT -> POT-RESCUE-CMOSworkshop_ThinStrips
Changed lines of the file:
@@
 EESchema Schematic File Version 2
+LIBS:CMOSworkshop_ThinStrips-rescue
 LIBS:power
 LIBS:device
@@
 LIBS:valves
 LIBS:CMOSworkshop-cache
-LIBS:4ms_JST_2x8
-LIBS:4ms-headers
-LIBS:4ms-ic
-LIBS:4ms-mech
-LIBS:4ms-passives
-LIBS:4ms-power
-LIBS:AudioBoardLib
-LIBS:EtherkitKicadLibrary
-LIBS:lm4880m
-LIBS:max97220
-LIBS:STM32F429_LQFP144
-LIBS:tpa6130
-LIBS:w_microcontrollers
-LIBS:wayne_and_layne_kicad_symbols
 LIBS:CMOSworkshop_ThinStrips-cache
 EELAYER 25 0
@@
 $EndComp
 $Comp
-L POT RV5
+L POT-RESCUE-CMOSworkshop_ThinStrips RV5
 U 1 1 58AD0187
 P 2650 1600
@@
 	1950 2800 1900 2800
 $Comp
-L POT RV6
+L POT-RESCUE-CMOSworkshop_ThinStrips RV6
 U 1 1 58AD144D
 P 3050 1600
@@
 	2350 2800 2300 2800
 $Comp
-L POT RV3
+L POT-RESCUE-CMOSworkshop_ThinStrips RV3
 U 1 1 58AD15FB
 P 1850 1600
@@
 	1100 2800 1050 2800
 $Comp
-L POT RV4
+L POT-RESCUE-CMOSworkshop_ThinStrips RV4
 U 1 1 58AD1645
 P 2250 1600
@@
 	1500 2800 1450 2800
 $Comp
-L POT RV1
+L POT-RESCUE-CMOSworkshop_ThinStrips RV1
 U 1 1 58AD20D3
 P 1050 1600
@@
 	1200 1850 1200 1600
 $Comp
-L POT RV2
+L POT-RESCUE-CMOSworkshop_ThinStrips RV2
 U 1 1 58AD20E4
 P 1450 1600

Commit message: changed touchpads to copper and adjusted for 2.54mm spacing
Parts:
- T1: renamed from U1; footprint Connect:touchpad3 -> DRCs parts:touchpadCopper
- T2: renamed from U2; footprint Connect:touchpad3 -> DRCs parts:touchpadCopper
- T3: renamed from U3; footprint Connect:touchpad3 -> DRCs parts:touchpadCopper
- T4: renamed from U4; footprint Connect:touchpad3 -> DRCs parts:touchpadCopper
- T5: renamed from U5; footprint Connect:touchpad3 -> DRCs parts:touchpadCopper
- T6: renamed from U6; footprint Connect:touchpad3 -> DRCs parts:touchpadCopper
Changed lines of the file:
@@
 	3850 3300 3800 3300
 $Comp
-L Touchpad U3
+L Touchpad T3
 U 1 1 58AD113B
 P 1850 2900
-F 0 "U3" H 1700 3000 60  0000 C CNN
+F 0 "T3" H 1700 3000 60  0000 C CNN
 F 1 "Touchpad" H 1850 2900 60  0000 C CNN
-F 2 "Connect:touchpad3" H 1850 2900 60  0001 C CNN
+F 2 "DRCs parts:touchpadCopper" H 1850 2900 60  0001 C CNN
 F 3 "" H 1850 2900 60  0001 C CNN
 	1    1850 2900
@@
 $EndComp
 $Comp
-L Touchpad U4
+L Touchpad T4
 U 1 1 58AD148E
 P 2250 2900
-F 0 "U4" H 2100 3000 60  0000 C CNN
+F 0 "T4" H 2100 3000 60  0000 C CNN
 F 1 "Touchpad" H 2250 2900 60  0000 C CNN
-F 2 "Connect:touchpad3" H 2250 2900 60  0001 C CNN
+F 2 "DRCs parts:touchpadCopper" H 2250 2900 60  0001 C CNN
 F 3 "" H 2250 2900 60  0001 C CNN
 	1    2250 2900
@@
 	4450 2900 4500 2900
 $Comp
-L Touchpad U1
+L Touchpad T1
 U 1 1 58AD163C
 P 1000 2900
-F 0 "U1" H 850 3000 60  0000 C CNN
+F 0 "T1" H 850 3000 60  0000 C CNN
 F 1 "Touchpad" H 1000 2900 60  0000 C CNN
-F 2 "Connect:touchpad3" H 1000 2900 60  0001 C CNN
+F 2 "DRCs parts:touchpadCopper" H 1000 2900 60  0001 C CNN
 F 3 "" H 1000 2900 60  0001 C CNN
 	1    1000 2900
@@
 	2250 2800 2250 3000
 $Comp
-L Touchpad U2
+L Touchpad T2
 U 1 1 58AD1686
 P 1400 2900
-F 0 "U2" H 1250 3000 60  0000 C CNN
+F 0 "T2" H 1250 3000 60  0000 C CNN
 F 1 "Touchpad" H 1400 2900 60  0000 C CNN
-F 2 "Connect:touchpad3" H 1400 2900 60  0001 C CNN
+F 2 "DRCs parts:touchpadCopper" H 1400 2900 60  0001 C CNN
 F 3 "" H 1400 2900 60  0001 C CNN
 	1    1400 2900
@@
 $EndComp
 $Comp
-L Touchpad U5
+L Touchpad T5
 U 1 1 58AD2193
 P 2600 2900
-F 0 "U5" H 2450 3000 60  0000 C CNN
+F 0 "T5" H 2450 3000 60  0000 C CNN
 F 1 "Touchpad" H 2600 2900 60  0000 C CNN
-F 2 "Connect:touchpad3" H 2600 2900 60  0001 C CNN
+F 2 "DRCs parts:touchpadCopper" H 2600 2900 60  0001 C CNN
 F 3 "" H 2600 2900 60  0001 C CNN
 	1    2600 2900
@@
 $EndComp
 $Comp
-L Touchpad U6
+L Touchpad T6
 U 1 1 58AD21A1
 P 3000 2900
-F 0 "U6" H 2850 3000 60  0000 C CNN
+F 0 "T6" H 2850 3000 60  0000 C CNN
 F 1 "Touchpad" H 3000 2900 60  0000 C CNN
-F 2 "Connect:touchpad3" H 3000 2900 60  0001 C CNN
+F 2 "DRCs parts:touchpadCopper" H 3000 2900 60  0001 C CNN
 F 3 "" H 3000 2900 60  0001 C CNN
 	1    3000 2900
