File: CMOSworkshop/power.sch (KiCad schematic (older format))
At the start: 11 parts, among them SW1 SW_DPDT_x2, U6 BAT9V

Commit message: updated pcb to accomodate 9v battery and made mixer circuit SMT due to space restrictions.  Spaced out knobs and touchpads for better ergonomics, and created touchpad footprints.
Parts:
- removed C14, C15, C17, C18, C19: 0.1uF, Capacitors_THT:C_Rect_L4.0mm_W2.5mm_P2.50mm, symbol C_Small
- removed C16: 0.1uF, Capacitors_THT:CP_Radial_D5.0mm_P2.50mm, symbol C_Small
- removed SW1: SW_DPDT_x2, 4ms-footprints:SPDT-SUB, symbol SW_DPDT_x2
- added S7: SPDT, 4ms-footprints:SPDT-SUB, symbol SPDT
- D2: footprint 4ms-footprints:D_SOD-123 -> Diodes_ThroughHole:Diode_DO-41_SOD81_Horizontal_RM10
- renumbered R18 to R13, U6 to U8
Connections:
- wire segments 18 -> 6
Changed lines of the file:
@@
 LIBS:contrib
 LIBS:valves
+LIBS:CMOSworkshop-cache
 LIBS:4ms_JST_2x8
 LIBS:4ms-headers
@@
 LIBS:w_microcontrollers
 LIBS:wayne_and_layne_kicad_symbols
-LIBS:74xgxx
-LIBS:ac-dc
-LIBS:actel
-LIBS:allegro
-LIBS:Altera
-LIBS:analog_devices
-LIBS:battery_management
-LIBS:bbd
-LIBS:brooktre
-LIBS:cmos_ieee
-LIBS:dc-dc
-LIBS:diode
-LIBS:elec-unifil
-LIBS:ESD_Protection
-LIBS:ftdi
-LIBS:gennum
-LIBS:graphic
-LIBS:hc11
-LIBS:ir
-LIBS:Lattice
-LIBS:logo
-LIBS:maxim
-LIBS:mechanical
-LIBS:microchip_dspic33dsc
-LIBS:microchip_pic10mcu
-LIBS:microchip_pic12mcu
-LIBS:microchip_pic16mcu
-LIBS:microchip_pic18mcu
-LIBS:microchip_pic32mcu
-LIBS:motor_drivers
-LIBS:motors
-LIBS:msp430
-LIBS:nordicsemi
-LIBS:nxp_armmcu
-LIBS:onsemi
-LIBS:Oscillators
-LIBS:Power_Management
-LIBS:powerint
-LIBS:pspice
-LIBS:references
-LIBS:relays
-LIBS:rfcom
-LIBS:sensors
-LIBS:silabs
-LIBS:stm8
-LIBS:stm32
-LIBS:supertex
-LIBS:switches
-LIBS:transf
-LIBS:ttl_ieee
-LIBS:video
-LIBS:wiznet
-LIBS:Worldsemi
-LIBS:Xicor
-LIBS:zetex
-LIBS:Zilog
-LIBS:CMOSworkshop-cache
+LIBS:CMOSworkshop_ThinStrips-cache
 EELAYER 25 0
 EELAYER END
 $Descr A4 11693 8268
 encoding utf-8
-Sheet 6 7
+Sheet 3 3
 Title ""
 Date ""
@@
 Wire Wire Line
 	7000 3450 7350 3450
-$Comp
-L C_Small C14
-U 1 1 589D6E67
-P 4450 3550
-F 0 "C14" H 4460 3620 50  0000 L CNN
-F 1 "0.1uF" H 4460 3470 50  0000 L CNN
-F 2 "Capacitors_THT:C_Rect_L4.0mm_W2.5mm_P2.50mm" H 4450 3550 50  0001 C CNN
-F 3 "" H 4450 3550 50  0000 C CNN
-	1    4450 3550
-	1    0    0    -1
-$EndComp
-$Comp
-L C_Small C15
-U 1 1 589D6EAB
-P 4650 3550
-F 0 "C15" H 4660 3620 50  0000 L CNN
-F 1 "0.1uF" H 4660 3470 50  0000 L CNN
-F 2 "Capacitors_THT:C_Rect_L4.0mm_W2.5mm_P2.50mm" H 4650 3550 50  0001 C CNN
-F 3 "" H 4650 3550 50  0000 C CNN
-	1    4650 3550
-	1    0    0    -1
-$EndComp
-$Comp
-L C_Small C16
-U 1 1 589D6EC1
-P 4850 3550
-F 0 "C16" H 4860 3620 50  0000 L CNN
-F 1 "0.1uF" H 4860 3470 50  0000 L CNN
-F 2 "Capacitors_THT:CP_Radial_D5.0mm_P2.50mm" H 4850 3550 50  0001 C CNN
-F 3 "" H 4850 3550 50  0000 C CNN
-	1    4850 3550
-	1    0    0    -1
-$EndComp
-$Comp
-L C_Small C17
-U 1 1 589D6ED9
-P 5050 3550
-F 0 "C17" H 5060 3620 50  0000 L CNN
-F 1 "0.1uF" H 5060 3470 50  0000 L CNN
-F 2 "Capacitors_THT:C_Rect_L4.0mm_W2.5mm_P2.50mm" H 5050 3550 50  0001 C CNN
-F 3 "" H 5050 3550 50  0000 C CNN
-	1    5050 3550
-	1    0    0    -1
-$EndComp
-$Comp
-L C_Small C18
-U 1 1 589D6EF5
-P 5250 3550
-F 0 "C18" H 5260 3620 50  0000 L CNN
-F 1 "0.1uF" H 5260 3470 50  0000 L CNN
-F 2 "Capacitors_THT:C_Rect_L4.0mm_W2.5mm_P2.50mm" H 5250 3550 50  0001 C CNN
-F 3 "" H 5250 3550 50  0000 C CNN
-	1    5250 3550
-	1    0    0    -1
-$EndComp
-$Comp
-L C_Small C19
-U 1 1 589D6F12
-P 5450 3550
-F 0 "C19" H 5460 3620 50  0000 L CNN
-F 1 "0.1uF" H 5460 3470 50  0000 L CNN
-F 2 "Capacitors_THT:C_Rect_L4.0mm_W2.5mm_P2.50mm" H 5450 3550 50  0001 C CNN
-F 3 "" H 5450 3550 50  0000 C CNN
-	1    5450 3550
-	1    0    0    -1
-$EndComp
 Wire Wire Line
 	4200 3800 7000 3800
@@
 VCC
 $Comp
-L VDD #PWR025
+L VDD #PWR09
 U 1 1 58A55182
 P 7350 3450
-F 0 "#PWR025" H 7350 3300 50  0001 C CNN
+F 0 "#PWR09" H 7350 3300 50  0001 C CNN
 F 1 "VDD" H 7350 3600 50  0000 C CNN
 F 2 "" H 7350 3450 50  0000 C CNN
@@
 $EndComp
 $Comp
-L GND #PWR026
+L GND #PWR010
 U 1 1 58A551A8
 P 7350 3650
-F 0 "#PWR026" H 7350 3400 50  0001 C CNN
+F 0 "#PWR010" H 7350 3400 50  0001 C CNN
 F 1 "GND" H 7350 3500 50  0000 C CNN
 F 2 "" H 7350 3650 50  0000 C CNN
@@
 Text GLabel 4200 3800 0    60   Input ~ 0
 GND
-Wire Wire Line
-	4450 3450 4450 3350
 Connection ~ 4450 3350
-Wire Wire Line
-	4650 3450 4650 3350
 Connection ~ 4650 3350
-Wire Wire Line
-	4850 3450 4850 3350
 Connection ~ 4850 3350
-Wire Wire Line
-	5050 3450 5050 3350
 Connection ~ 5050 3350
-Wire Wire Line
-	5250 3450 5250 3350
 Connection ~ 5250 3350
-Wire Wire Line
-	5450 3450 5450 3350
 Connection ~ 5450 3350
-Wire Wire Line
-	4450 3650 4450 3800
 Connection ~ 4450 3800
-Wire Wire Line
-	4650 3650 4650 3800
 Connection ~ 4650 3800
-Wire Wire Line
-	4850 3650 4850 3800
 Connection ~ 4850 3800
-Wire Wire Line
-	5050 3650 5050 3800
 Connection ~ 5050 3800
-Wire Wire Line
-	5250 3650 5250 3800
 Connection ~ 5250 3800
-Wire Wire Line
-	5450 3650 5450 3800
 Connection ~ 5450 3800
 $Comp
-L BAT9V U6
+L BAT9V U8
 U 1 1 58A8CEFA
 P 9700 3850
-F 0 "U6" H 9750 4550 60  0000 C CNN
+F 0 "U8" H 9750 4550 60  0000 C CNN
 F 1 "BAT9V" H 9750 3700 60  0000 C CNN
 F 2 "Battery_Holders:Battery_Conn" H 9700 3850 60  0001 C CNN
@@
 $EndComp
 $Comp
-L VDD #PWR027
+L VDD #PWR011
 U 1 1 58A8CF8F
-P 8500 3200
-F 0 "#PWR027" H 8500 3050 50  0001 C CNN
-F 1 "VDD" H 8500 3350 50  0000 C CNN
-F 2 "" H 8500 3200 50  0000 C CNN
-F 3 "" H 8500 3200 50  0000 C CNN
-	1    8500 3200
+P 8400 3200
+F 0 "#PWR011" H 8400 3050 50  0001 C CNN
+F 1 "VDD" H 8400 3350 50  0000 C CNN
+F 2 "" H 8400 3200 50  0000 C CNN
+F 3 "" H 8400 3200 50  0000 C CNN
+	1    8400 3200
 	1    0    0    -1
 $EndComp
 $Comp
-L GND #PWR028
+L GND #PWR012
 U 1 1 58A8CFAF
 P 9200 3850
-F 0 "#PWR028" H 9200 3600 50  0001 C CNN
+F 0 "#PWR012" H 9200 3600 50  0001 C CNN
 F 1 "GND" H 9200 3700 50  0000 C CNN
 F 2 "" H 9200 3850 50  0000 C CNN
@@
 F 0 "D2" H 9050 3400 50  0000 C CNN
 F 1 "B140HW-7" H 9050 3200 50  0000 C CNN
-F 2 "4ms-footprints:D_SOD-123" H 9050 3125 50  0001 C CNN
+F 2 "Diodes_ThroughHole:Diode_DO-41_SOD81_Horizontal_RM10" H 9050 3125 50  0001 C CNN
 F 3 "" H 9050 3300 50  0001 C CNN
 	1    9050 3300
 	1    0    0    -1
-$EndComp
-$Comp
-L SW_DPDT_x2 SW1
-U 1 1 58A8DB53
-P 8700 3300
-F 0 "SW1" H 8700 3470 50  0000 C CNN
-F 1 "SW_DPDT_x2" H 8900 3300 50  0000 C CNN
-F 2 "4ms-footprints:SPDT-SUB" H 8700 3300 50  0001 C CNN
-F 3 "" H 8700 3300 50  0000 C CNN
-	1    8700 3300
-	-1   0    0    1
 $EndComp
 $Comp
@@
 $EndComp
 $Comp
-L GND #PWR029
+L GND #PWR013
 U 1 1 58A8DCBF
 P 7750 4250
-F 0 "#PWR029" H 7750 4000 50  0001 C CNN
+F 0 "#PWR013" H 7750 4000 50  0001 C CNN
 F 1 "GND" H 7750 4100 50  0000 C CNN
 F 2 "" H 7750 4250 50  0000 C CNN
@@
 $EndComp
 $Comp
-L R_Small R18
+L R_Small R13
 U 1 1 58A8DD9C
 P 7750 4150
-F 0 "R18" H 7780 4170 50  0000 L CNN
+F 0 "R13" H 7780 4170 50  0000 L CNN
 F 1 "1K" H 7780 4110 50  0000 L CNN
 F 2 "4ms-footprints:R-TH" H 7750 4150 50  0001 C CNN
@@
 $EndComp
 $Comp
-L VDD #PWR030
+L VDD #PWR014
 U 1 1 58A8DFC4
 P 7750 3750
-F 0 "#PWR030" H 7750 3600 50  0001 C CNN
+F 0 "#PWR014" H 7750 3600 50  0001 C CNN
 F 1 "VDD" H 7750 3900 50  0000 C CNN
 F 2 "" H 7750 3750 50  0000 C CNN
@@
 	1    0    0    -1
 $EndComp
+$Comp
+L SPDT S7
+U 1 1 58AD2C37
+P 8650 3300
+F 0 "S7" H 8640 3590 50  0000 C CNN
+F 1 "SPDT" H 8650 3500 50  0000 C CNN
+F 2 "4ms-footprints:SPDT-SUB" H 8650 3300 60  0001 C CNN
+F 3 "" H 8650 3300 60  0000 C CNN
+	1    8650 3300
+	-1   0    0    1
+$EndComp
 $EndSCHEMATC

Commit message: updated mixer schematic, added 9v battery holder and laid out components.
Parts:
- U8: footprint Battery_Holders:Battery_Conn -> DRCs parts:9V_BatteryHolder_Keystone
Changed lines of the file:
@@
 F 0 "U8" H 9750 4550 60  0000 C CNN
 F 1 "BAT9V" H 9750 3700 60  0000 C CNN
-F 2 "Battery_Holders:Battery_Conn" H 9700 3850 60  0001 C CNN
+F 2 "DRCs parts:9V_BatteryHolder_Keystone" H 9700 3850 60  0001 C CNN
 F 3 "" H 9700 3850 60  0000 C CNN
 	1    9700 3850

Commit message: added traces for mixer circuit and made small connection in hp mixer
Parts:
- D1: symbol LED -> LED-RESCUE-CMOSworkshop_ThinStrips
- R13: symbol R_Small -> R_Small-RESCUE-CMOSworkshop_ThinStrips
Changed lines of the file:
@@
 EESchema Schematic File Version 2
+LIBS:CMOSworkshop_ThinStrips-rescue
 LIBS:power
 LIBS:device
@@
 LIBS:valves
 LIBS:CMOSworkshop-cache
-LIBS:4ms_JST_2x8
-LIBS:4ms-headers
-LIBS:4ms-ic
-LIBS:4ms-mech
-LIBS:4ms-passives
-LIBS:4ms-power
-LIBS:AudioBoardLib
-LIBS:EtherkitKicadLibrary
-LIBS:lm4880m
-LIBS:max97220
-LIBS:STM32F429_LQFP144
-LIBS:tpa6130
-LIBS:w_microcontrollers
-LIBS:wayne_and_layne_kicad_symbols
 LIBS:CMOSworkshop_ThinStrips-cache
 EELAYER 25 0
@@
 $EndComp
 $Comp
-L LED D1
+L LED-RESCUE-CMOSworkshop_ThinStrips D1
 U 1 1 58A8DBDC
 P 7750 3900
@@
 $EndComp
 $Comp
-L R_Small R13
+L R_Small-RESCUE-CMOSworkshop_ThinStrips R13
 U 1 1 58A8DD9C
 P 7750 4150
