File: CMOSworkshop/CMOSworkshop_ThinStrips.kicad_pcb (KiCad board)
At the start: 2 copper layers, 160.5 x 65.6 mm, 68 parts, among them J1 JACK_STEREO, P1 CONN_01X03, P10 CONN_01X02, P11 CONN_01X03, P12 CONN_01X02, P13 CONN_01X03, P14 CONN_01X02, P15 CONN_01X03, P16 CONN_01X02, P17 CONN_01X02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

Commit message: pushing ahead of work comp
Parts:
- removed P10, P6, P8: CONN_01X02, EtherkitKicadLibrary:Pin_Header_Straight_1x02
- removed the P3 at (126.9, 108.0)
- removed P5: CONN_01X03, 4ms-footprints:Pin_Header_Straight_1x03
- removed the S4 at (189.6, 142.8)
- removed U3: Touchpad, Connect:touchpad3
- added G***: LOGO, CMOSworkshop:geotouchpoint, F.Cu at (141.0, 88.0)
- added P11: CONN_01X03, 4ms-footprints:Pin_Header_Straight_1x03, F.Cu at (157.5, 106.7)
- added P11: CONN_01X03, 4ms-footprints:Pin_Header_Straight_1x03, F.Cu at (157.5, 109.2)
- added P11: CONN_01X03, 4ms-footprints:Pin_Header_Straight_1x03, F.Cu at (147.3, 106.7)
- added P11: CONN_01X03, 4ms-footprints:Pin_Header_Straight_1x03, F.Cu at (147.3, 109.2)
- added P11: CONN_01X03, 4ms-footprints:Pin_Header_Straight_1x03, F.Cu at (137.2, 109.2)
- added P11: CONN_01X03, 4ms-footprints:Pin_Header_Straight_1x03, F.Cu at (137.2, 106.7)
- added P11: CONN_01X03, 4ms-footprints:Pin_Header_Straight_1x03, F.Cu at (114.3, 109.2)
- added P3: CONN_01X03, 4ms-footprints:Pin_Header_Straight_1x03, F.Cu at (104.1, 106.7)
- added P3: CONN_01X03, 4ms-footprints:Pin_Header_Straight_1x03, F.Cu at (104.1, 104.1)
- added P3: CONN_01X03, 4ms-footprints:Pin_Header_Straight_1x03, F.Cu at (104.1, 109.2)
- added P3: CONN_01X03, 4ms-footprints:Pin_Header_Straight_1x03, F.Cu at (124.5, 104.1)
- added P3: CONN_01X03, 4ms-footprints:Pin_Header_Straight_1x03, F.Cu at (124.5, 106.7)
- added P3: CONN_01X03, 4ms-footprints:Pin_Header_Straight_1x03, F.Cu at (124.5, 109.2)
- added REF**: 2.54mm_solder_pads, DRCs parts:2.54mm_5x5_pads, F.Cu at (193.0, 134.6)
- RV2, RV3, RV6: value POT -> 100K
- U1, U2, U4, U5, U6: footprint Connect:touchpad3 -> DRCs parts:touchpad3(2.54mm)
- moved P16 33.0 mm to (190.7, 160.0)
- moved P17 33.0 mm to (213.1, 159.8)
- moved S2 33.0 mm to (220.2, 175.6)
- moved S4 33.0 mm to (204.8, 175.6)
- moved S5 33.0 mm to (197.4, 170.6)
- moved P14 33.0 mm to (220.6, 159.8)
- moved P16 33.0 mm to (205.9, 159.8)
- moved P17 33.0 mm to (197.9, 160.0)
- moved P19 33.0 mm to (229.0, 159.6)
- moved S5 33.0 mm to (212.6, 170.4)
- moved S6 33.0 mm to (228.1, 170.1)
- moved U4 4.13 mm to (152.4, 104.1)
- moved RV2 3.99 mm to (127.0, 87.0)
- moved U5 3.39 mm to (162.6, 96.4)
- moved RV3 1.72 mm to (106.7, 87.0)
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Routing:
- net Net-(P3-Pad3): track 0.00 -> 29.3 mm
- net Net-(P3-Pad2): track 0.00 -> 29.3 mm
- net Net-(P3-Pad1): track 0.00 -> 29.3 mm
- net Net-(P11-Pad2): track 0.00 -> 24.5 mm
- net Net-(P11-Pad3): track 0.00 -> 12.8 mm
- net Net-(P11-Pad1): track 0.00 -> 12.8 mm
- net Net-(P10-Pad2): track 0.00 -> 11.5 mm
- net Net-(P10-Pad1): track 0.00 -> 11.5 mm
- net Net-(P6-Pad2): track 0.00 -> 11.4 mm
- net Net-(P8-Pad2): track 0.00 -> 3.74 mm
- net Net-(P8-Pad1): track 0.00 -> 3.74 mm
- net (no net): track 0.00 -> 2.54 mm
